Commit message: feat: add fixed frame

File: urdf/umaru.xacro (robot description, xacro)
@@ -28,4 +28,16 @@
     </joint>
   </xacro:macro>
+  <xacro:macro name="m_joint_fixed" params="joint_name parent child xyz rpy">
+    <joint name="${joint_name}" type="fixed">
+      <parent link="${parent}"/>
+      <child link="${child}"/>
+      <origin xyz="${xyz}" rpy="${rpy}"/>
+    </joint>
+  </xacro:macro>
+  <xacro:macro name="m_frame" params="frame_name">
+    <link name="${frame_name}">
+    <origion xyz="0 0 0" rpy="0 0 0"></origion>
+    </link>
+  </xacro:macro>
   <material name="black">
     <color rgba="0.25 0.25 0.25 1"/>
@@ -38,4 +50,6 @@
   </material>
   <link name="base_link"/>
+  <xacro:m_frame frame_name="odom"/>
+  <xacro:m_joint joint_name="odom_joint" parent="base_link" child="odom" xyz="0 0 0" rpy="0 0 0" lower="0" upper="0"/>
   <!-- BODY -->
   <xacro:m_link link_name="body" xyz="${0*world_scale} ${0*world_scale} ${0*world_scale}" rpy="${pi/2} 0 0" mesh="Body" color="black"/>
@@ -113,3 +127,13 @@
   <xacro:m_joint joint_name="neck_pitch" parent="neck" child="head"
                   xyz="${0.175*world_scale} ${0*world_scale} ${0*world_scale}" rpy="${pi/2} ${pi} ${pi/2}" lower="${pi/-2}" upper="${pi/8}"/>
+  <!-- FRAMES -->
+  <xacro:m_frame frame_name="camera"/>
+  <xacro:m_joint joint_name="camera_joint" parent="head" child="camera"
+                        xyz="${0*world_scale} ${0.1*world_scale} ${0.2*world_scale}" rpy="0 0 0" lower="0" upper="0"/>
+  <xacro:m_frame frame_name="right_foot_frame"/>
+  <xacro:m_joint joint_name="right_foot_joint" parent="right_foot" child="right_foot_frame"
+                        xyz="${0*world_scale} ${0*world_scale} ${0.2*world_scale}" rpy="0 0 0" lower="0" upper="0"/>
+  <xacro:m_frame frame_name="left_foot_frame"/>
+  <xacro:m_joint joint_name="left_foot_joint" parent="left_foot" child="left_foot_frame"
+                        xyz="${0*world_scale} ${0*world_scale} ${0.2*world_scale}" rpy="0 0 0" lower="0" upper="0"/>
 </robot>

Commit message: fix: hip yaw direction

File: urdf/umaru.xacro (robot description, xacro)
@@ -51,12 +51,8 @@
   <link name="base_link"/>
   <xacro:m_frame frame_name="odom"/>
-  <xacro:m_joint joint_name="odom_joint" parent="base_link" child="odom" xyz="0 0 0" rpy="0 0 0" lower="0" upper="0"/>
+  <xacro:m_joint_fixed joint_name="odom_joint" parent="base_link" child="odom" xyz="0 0 0" rpy="0 0 0"/>
   <!-- BODY -->
   <xacro:m_link link_name="body" xyz="${0*world_scale} ${0*world_scale} ${0*world_scale}" rpy="${pi/2} 0 0" mesh="Body" color="black"/>
-  <joint name="body_joint" type="fixed">
-    <parent link="base_link"/>
-    <child link="body"/>
-    <origin xyz="0 0 ${2.75*world_scale}" rpy="0 0 0"/>
-  </joint>
+  <xacro:m_joint joint_name="body_joint" parent="odom" child="body" xyz="0 0 ${2.75 * world_scale}" rpy="0 0 0" lower="0" upper="0"/>
   <!-- HEAD LINK -->
   <xacro:m_link link_name="neck" xyz="${0*world_scale} ${-0.092*world_scale} ${-0.065*world_scale}" rpy="${pi/2} ${pi/2} 0" mesh="Neck" color="light_gray"/>
@@ -99,7 +95,7 @@
   <!-- LEG JOINTS (ID 7 - 18) -->
   <xacro:m_joint joint_name="right_hip_yaw" parent="body" child="right_groin"
-                  xyz="${-0.238*world_scale} ${-0.2475*world_scale} ${-0.68*world_scale}" rpy="0 ${pi/-2} 0" lower="${pi/-4}" upper="${pi/2}"/>
+                  xyz="${-0.238*world_scale} ${-0.2475*world_scale} ${-0.68*world_scale}" rpy="0 ${pi/-2} 0" lower="${pi/-2}" upper="${pi/4}"/>
   <xacro:m_joint joint_name="left_hip_yaw" parent="body" child="left_groin"
-                  xyz="${-0.238*world_scale} ${0.2475*world_scale} ${-0.68*world_scale}" rpy="0 ${pi/-2} 0" lower="${pi/-2}" upper="${pi/4}"/>
+                  xyz="${-0.238*world_scale} ${0.2475*world_scale} ${-0.68*world_scale}" rpy="0 ${pi/-2} 0" lower="${pi/-4}" upper="${pi/2}"/>
   <xacro:m_joint joint_name="right_hip_roll" parent="right_groin" child="right_buttock"
                   xyz="${-0.185*world_scale} ${0*world_scale} ${0.135*world_scale}" rpy="0 ${pi/-2} 0" lower="${pi/-4}" upper="${pi/2}"/>
