Commit message: feat: progress until hip pitch

File: urdf/double_crank.xacro (robot description, xacro)
@@ -45,4 +45,13 @@
     </joint>
   </xacro:macro>
+  <xacro:macro name="m_joint_mimic" params="joint_name parent child xyz rpy lower upper mimic mult">
+    <joint name="${joint_name}" type="revolute">
+      <parent link="${parent}"/>
+      <child link="${child}"/>
+      <origin xyz="${xyz}" rpy="${rpy}"/>
+      <mimic joint="${mimic}" multiplier="${mult}" offset="0"/>
+      <limit effort="1000" lower="${lower}" upper="${upper}" velocity="1"/>
+    </joint>
+  </xacro:macro>
   <xacro:macro name="m_joint_fixed" params="joint_name parent child xyz rpy">
     <joint name="${joint_name}" type="fixed">
@@ -85,5 +94,7 @@
   <!-- RIGHT LEG LINK -->
   <xacro:m_link_leg link_name="right_groin" xyz="${-0.01*world_scale} ${-0.235*world_scale} ${0.375*world_scale}" rpy="0 ${pi/2} ${pi/2}" mesh="Groin" color="light_gray"/>
-  <xacro:m_link_leg link_name="right_upper_hip" xyz="${-0.355*world_scale} ${0.235*world_scale} ${-0.19*world_scale}" rpy="${pi/2} 0 0" mesh="Upper_Hip" color="light_gray"/>
+  <xacro:m_link_leg link_name="right_hip" xyz="${-0.355*world_scale} ${0.235*world_scale} ${-0.13*world_scale}" rpy="${pi/2} 0 0" mesh="Upper_Hip" color="light_gray"/>
+  <xacro:m_link_leg link_name="right_hip_front_crank" xyz="${0*world_scale} ${0.0525*world_scale} ${0.255*world_scale}" rpy="${pi/2} 0 ${pi/-2}" mesh="Upper_Front_Crank" color="black"/>
+  <xacro:m_link_leg link_name="right_hip_behind_crank" xyz="${-0.165*world_scale} ${-0.09*world_scale} ${0.305*world_scale}" rpy="${pi/2} 0 ${pi/-2}" mesh="Upper_Behind_Crank" color="black"/>
   <!-- <xacro:m_link link_name="right_groin" xyz="${-0.415*world_scale} ${-0.235*world_scale} ${-0.05*world_scale}" rpy="${pi/-2} ${pi/-2} 0" mesh="Groin" color="light_gray"/>
   <xacro:m_link link_name="right_buttock" xyz="${-0.18*world_scale} ${-0.235*world_scale} ${0.23*world_scale}" rpy="${pi/-2} 0 0" mesh="Buttock" color="light_gray"/>
@@ -94,4 +105,7 @@
   <!-- LEFT LEG LINK -->
   <xacro:m_link_leg link_name="left_groin" xyz="${-0.01*world_scale} ${-0.235*world_scale} ${0.375*world_scale}" rpy="0 ${pi/2} ${pi/2}" mesh="Groin" color="light_gray"/>
+  <xacro:m_link_leg link_name="left_hip" xyz="${-0.355*world_scale} ${0.235*world_scale} ${-0.13*world_scale}" rpy="${pi/2} 0 0" mesh="Upper_Hip" color="light_gray"/>
+  <xacro:m_link_leg link_name="left_hip_front_crank" xyz="${0*world_scale} ${0.0525*world_scale} ${0.255*world_scale}" rpy="${pi/2} 0 ${pi/-2}" mesh="Upper_Front_Crank" color="black"/>
+  <xacro:m_link_leg link_name="left_hip_behind_crank" xyz="${-0.165*world_scale} ${-0.09*world_scale} ${0.305*world_scale}" rpy="${pi/2} 0 ${pi/-2}" mesh="Upper_Behind_Crank" color="black"/>
   <!-- <xacro:m_link link_name="left_groin" xyz="${-0.415*world_scale} ${-0.235*world_scale} ${-0.05*world_scale}" rpy="${pi/-2} ${pi/-2} 0" mesh="Groin" color="light_gray"/>
   <xacro:m_link link_name="left_buttock" xyz="${-0.18*world_scale} ${-0.235*world_scale} ${0.23*world_scale}" rpy="${pi/-2} 0 0" mesh="Buttock" color="light_gray"/>
@@ -118,6 +132,18 @@
   <xacro:m_joint joint_name="left_hip_yaw" parent="body" child="left_groin"
                   xyz="${-0.238*world_scale} ${0.2475*world_scale} ${-0.68*world_scale}" rpy="0 ${pi/-2} 0" lower="${pi/-4}" upper="${pi/2}"/>
-  <xacro:m_joint joint_name="right_hip_roll" parent="right_groin" child="right_upper_hip"
-                  xyz="${-0.15*world_scale} ${0*world_scale} ${0*world_scale}" rpy="0 ${pi/-2} 0" lower="${pi/-4}" upper="${pi/2}"/>
+  <xacro:m_joint joint_name="right_hip_roll" parent="right_groin" child="right_hip"
+                  xyz="${-0.14*world_scale} ${0*world_scale} ${0*world_scale}" rpy="0 ${pi/-2} 0" lower="${pi/-4}" upper="${pi/2}"/>
+  <xacro:m_joint joint_name="left_hip_roll" parent="left_groin" child="left_hip"
+                  xyz="${-0.14*world_scale} ${0*world_scale} ${0*world_scale}" rpy="0 ${pi/-2} 0" lower="${pi/-2}" upper="${pi/4}"/>
+  <xacro:m_joint joint_name="right_hip_pitch" parent="right_hip" child="right_hip_front_crank"
+                  xyz="${-0.02*world_scale} ${0*world_scale} ${0.14*world_scale}" rpy="0 0 ${pi/2}" lower="${pi/-2}" upper="${pi/6}"/>
+  <xacro:m_joint joint_name="left_hip_pitch" parent="left_hip" child="left_hip_front_crank"
+                  xyz="${-0.02*world_scale} ${0*world_scale} ${0.14*world_scale}" rpy="0 0 ${pi/2}" lower="${pi/-2}" upper="${pi/6}"/>
+  <xacro:m_joint_mimic joint_name="right_hip_pitch_mimic" parent="right_hip" child="right_hip_behind_crank"
+                  xyz="${0.1775*world_scale} ${0*world_scale} ${0.26*world_scale}" rpy="0 0 ${pi/2}" lower="${pi/-2}" upper="${pi/6}"
+                  mimic="right_hip_pitch" mult="1"/>
+  <xacro:m_joint_mimic joint_name="left_hip_pitch_mimic" parent="left_hip" child="left_hip_behind_crank"
+                  xyz="${0.1775*world_scale} ${0*world_scale} ${0.26*world_scale}" rpy="0 0 ${pi/2}" lower="${pi/-2}" upper="${pi/6}"
+                  mimic="left_hip_pitch" mult="1"/>
   <!-- <xacro:m_joint joint_name="right_hip_yaw" parent="body" child="right_groin"
                   xyz="${-0.238*world_scale} ${-0.2475*world_scale} ${-0.68*world_scale}" rpy="0 ${pi/-2} 0" lower="${pi/-2}" upper="${pi/4}"/>
